File: lightspeakers.brd (EAGLE design)
At the start: 50 x 50 mm, 38 parts, among them IC1 LM1117 5V Regulator, IC3 OPAMP-DUALU, J1 POWER_JACKPTH, J2 1X2-3.5MM, Q1 2N2222, U1 RELAY-SOLIDSTATEPTH, U2 Audio Jack

Commit message: updates
Parts:
- removed IC3: OPAMP-DUALU, SparkFun:SO08
- removed J2: 1X2-3.5MM, adafruit:1X2-3.5MM
- added IC2: LM324D, linear:SO14
- added JP1: (no value), SparkFun:SCREWTERMINAL-5MM-2
- C6: device SparkFun:0402-CAP -> SparkFun:0603-CAP
- D1: device SparkFun:SMA-DIODE -> SparkFun:DIODE-1N4001
- R3: value 2.2k -> 1k
- S1: device SparkFun:SWITCH-SPDT-SMD -> SparkFun:SWITCH-SPDT
- moved U$2 19.0 mm to (22.9, 2.54)
- moved R12 16.9 mm to (31.8, 19.1)
- moved R14 16.3 mm to (28.2, 21.6)
- moved R6 15.1 mm to (34.3, 19.1)
- moved D1 14.2 mm to (38.1, 16.5), turned to 90 degrees
- moved R13 11.6 mm to (24.6, 21.6), turned to 0 degrees
- moved C4 6.67 mm to (20.8, 21.6)
- moved R10 4.84 mm to (42.5, 11.4), turned to 180 degrees
- moved C6 4.58 mm to (17.8, 15.2), turned to 180 degrees
- moved R11 4.50 mm to (42.5, 9.02), turned to 0 degrees
- moved C8 4.02 mm to (18.3, 29.0)
- moved R1 3.59 mm to (42.5, 15.2)
- moved C9 3.25 mm to (24.1, 41.4), turned to 90 degrees
- moved IC1 2.87 mm to (18.9, 35.1)
- moved C2 2.54 mm to (34.3, 11.4)
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Connections:
- removed net N$3: J2.1, U1.2
- new net N$27: C4.1, IC2.1, IC2.2, IC2.6, IC2.7, JP2.2, JP3.1
- new net N$28: IC2.3, U2.RING
- new net N$29: JP1.2, U1.1
- net GND: now also IC2.11, IC2.9; no longer IC3.3, IC3.4
- net N$10: now also IC2.10; no longer IC3.2
- net N$17: now also IC2.13; no longer IC3.5
- net N$18: now also IC2.14; no longer IC3.7
- net N$19: now also IC2.12; no longer IC3.6
- net N$22: now also IC2.5; no longer C4.1, JP2.2, JP3.1, U2.RING
- net N$4: now also JP1.1, U1.2; no longer J2.2, U1.1
- net N$9: now also IC2.8; no longer IC3.1
- net VCC: now also IC2.4; no longer IC3.8
Routing:
- net N$27: track 0.00 -> 53.7 mm, vias 0 -> 1
- net N$22: track 63.0 -> 17.8 mm
- net GND: track 54.9 -> 38.0 mm
- net N$8: track 29.8 -> 14.9 mm, vias 1 -> 0
- net VCC: track 30.2 -> 17.1 mm
- net N$28: track 0.00 -> 12.9 mm
- net N$29: track 0.00 -> 10.6 mm
- net N$3: track 10.2 -> 1.27 mm
- net N$9: track 20.4 -> 13.4 mm
- net N$4: track 11.4 -> 7.14 mm
- net N$1: track 18.5 -> 15.0 mm
- net N$19: track 14.7 -> 11.3 mm
- net N$12: track 9.82 -> 12.9 mm
- net N$2: track 11.0 -> 13.8 mm
- net N$21: track 19.7 -> 17.8 mm
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
Commit message: Finished PCB, added fuse, sending out
Parts:
- added F1: FUSE, SparkFun:20MMX5MMFUSE
- C8, C9: device SparkFun:EIA6032 -> SparkFun:CPOL-RADIAL-10UF-25V
- moved Q1 24.1 mm to (21.6, 27.9)
- moved C9 21.9 mm to (14.7, 21.6), turned to 0 degrees
- moved U1 10.2 mm to (28.6, 38.1)
- moved R3 8.13 mm to (28.2, 24.1), turned to 180 degrees
- moved C8 3.64 mm to (14.7, 28.2), turned to 180 degrees
- moved S1 1.27 mm to (2.96, 25.4)
- moved J1 1.27 mm to (-3.17, 36.8)
Connections:
- new net N$30: F1.P$2, JP1.1
- net GND: now also C8.2, C9.2; no longer C8.P$2, C9.P$2
- net N$21: now also C8.1; no longer C8.P$1
- net N$4: now also F1.P$1; no longer JP1.1
- net VCC: now also C9.1; no longer C9.P$1
Routing:
- net N$1: track 15.0 -> 33.3 mm, vias 0 -> 1
- net N$30: track 0.00 -> 12.9 mm
- net N$29: track 10.6 -> 21.6 mm
- net N$2: track 13.8 -> 23.9 mm
- net N$8: track 14.9 -> 20.1 mm
- net GND: track 38.0 -> 33.1 mm, vias 8 -> 6
- net N$4: track 7.14 -> 10.6 mm
- net N$18: track 23.9 -> 21.3 mm, vias 2 -> 1
- net N$5: track 10.2 -> 7.97 mm, vias 1 -> 0
- net N$21: track 17.8 -> 16.3 mm
- net N$3: track 1.27 -> 0.00 mm
Other:
- board text added: "D53497"
