File: lightspeakers.sch (EAGLE design)
At the start: 38 parts, among them IC1 LM1117 5V Regulator, IC3 OPAMP-DUALU, J1 POWER_JACKPTH, J2 1X2-3.5MM, Q1 2N2222, U1 RELAY-SOLIDSTATEPTH, U2 Audio Jack

Commit message: updates
Parts:
- removed IC3: OPAMP-DUALU, SparkFun:OPAMP-DUALU
- removed J2: 1X2-3.5MM, adafruit:1X2-3.5MM
- added IC2: LM324D, linear:LM324D
- added JP1: (no value), SparkFun:M025MM
- C6: device SparkFun:CAP0402-CAP -> SparkFun:CAP0603-CAP
- D1: device SparkFun:DIODESMA -> SparkFun:DIODEPTH
- R3: value 2.2k -> 1k
- S1: device SparkFun:SWITCH-SPSTSMD2 -> SparkFun:SWITCH-SPSTPTH
Connections:
- removed net N$3: J2.1, U1.T2
- new net N$27: C4.1, IC2A.-IN, IC2A.OUT, IC2B.-IN, IC2B.OUT, JP2.2, JP3.1
- new net N$28: IC2A.+IN, U2.RIGHT
- new net N$29: JP1.2, U1.T1
- net GND: now also IC2C.-IN, IC2P.V-; no longer IC3A.+IN, IC3A.V-
- net N$10: now also IC2C.+IN; no longer IC3A.-IN
- net N$17: now also IC2D.-IN; no longer IC3B.+IN
- net N$18: now also IC2D.OUT; no longer IC3B.OUT
- net N$19: now also IC2D.+IN; no longer IC3B.-IN
- net N$22: now also IC2B.+IN; no longer C4.1, JP2.2, JP3.1, U2.RIGHT
- net N$4: now also JP1.1, U1.T2; no longer J2.2, U1.T1
- net N$9: now also IC2C.OUT; no longer IC3A.OUT
- net VCC: now also IC2P.V+; no longer IC3A.V+
Other:
- moved on the sheet: U2

Commit message: Finished PCB, added fuse, sending out
Parts:
- added F1: FUSE, SparkFun:FUSE
- C8, C9: device SparkFun:CAP_POL6032 -> SparkFun:CAP_POLPTH2
Connections:
- new net N$30: F1.2, JP1.1
- net N$4: now also F1.1; no longer JP1.1
Changed lines of the file:
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@@
 <part name="J1" library="SparkFun" deviceset="POWER_JACK" device="PTH"/>
 <part name="IC1" library="SparkFun" deviceset="V_REG_LM1117" device="SOT223" value="LM1117 5V Regulator"/>
-<part name="C8" library="SparkFun" deviceset="CAP_POL" device="6032" value="10uF"/>
-<part name="C9" library="SparkFun" deviceset="CAP_POL" device="6032" value="10uF"/>
+<part name="C8" library="SparkFun" deviceset="CAP_POL" device="PTH2" value="10uF"/>
+<part name="C9" library="SparkFun" deviceset="CAP_POL" device="PTH2" value="10uF"/>
 <part name="GND12" library="SparkFun" deviceset="GND" device=""/>
 <part name="GND13" library="SparkFun" deviceset="GND" device=""/>
@@
 <part name="IC2" library="linear" deviceset="LM324" device="D"/>
 <part name="JP1" library="SparkFun" deviceset="M02" device="5MM"/>
+<part name="F1" library="SparkFun" deviceset="FUSE" device=""/>
 </parts>
 <sheets>
@@
 <instance part="IC2" gate="D" x="83.82" y="88.9"/>
 <instance part="IC2" gate="C" x="144.78" y="73.66"/>
+<instance part="F1" gate="G$1" x="223.52" y="119.38"/>
 </instances>
 <busses>
@@
 <net name="N$4" class="0">
 <segment>
-<pinref part="JP1" gate="G$1" pin="1"/>
 <pinref part="U1" gate="G$1" pin="T2"/>
 <wire x1="218.44" y1="96.52" x2="210.82" y2="96.52" width="0.1524" layer="91"/>
-<wire x1="236.22" y1="116.84" x2="210.82" y2="116.84" width="0.1524" layer="91"/>
-<wire x1="210.82" y1="116.84" x2="210.82" y2="96.52" width="0.1524" layer="91"/>
-</segment>
-</net>
+<wire x1="210.82" y1="119.38" x2="210.82" y2="96.52" width="0.1524" layer="91"/>
+<pinref part="F1" gate="G$1" pin="1"/>
+<wire x1="213.36" y1="119.38" x2="210.82" y2="119.38" width="0.1524" layer="91"/>
+</segment>
+</net>
+<net name="N$30" class="0">
+<segment>
+<pinref part="F1" gate="G$1" pin="2"/>
+<pinref part="JP1" gate="G$1" pin="1"/>
+<wire x1="233.68" y1="119.38" x2="236.22" y2="119.38" width="0.1524" layer="91"/>
+<wire x1="236.22" y1="119.38" x2="236.22" y2="116.84" width="0.1524" layer="91"/>
+</segment>
+</net>
